File: 04_servo_tester/servo_tester.kicad_pcb (KiCad board)
At the start: 2 copper layers, 32.7 x 29.6 mm, 10 parts, among them J1 Conn_01x02_Pin, J2 Conn_01x03_Pin, U1 NE555P

Commit message: GND Zone Updated
Routing:
- added copper zone on B.Cu, net GND
Changed lines of the file:
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@@
 		(net 4)
 		(net_name "GND")
-		(layer "F.Cu")
+		(layers "F.Cu" "B.Cu")
 		(hatch edge 0.5)
 		(connect_pads
